File: PCB_Casque/PCB_Casque.kicad_sch (KiCad schematic)
At the start: 0 parts

Commit message: ajout du PCB version final + elt du design
Other:
- added sheet trou_fixation (trou_fixation.kicad_sch)
- sheet ESP23_s3_mini_1_N8 ports: added DN, DP; removed D+, D-
- sheet USB_C ports: added DN, DP; removed D+, D-
Changed lines of the file:
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@@
 			)
 		)
-		(pin "D+" bidirectional
+		(pin "DP" bidirectional
 			(at 48.26 58.42 270)
 			(effects
@@
 			)
 		)
-		(pin "D-" bidirectional
+		(pin "DN" bidirectional
 			(at 45.72 58.42 270)
 			(effects
@@
 			)
 		)
-		(pin "D+" bidirectional
+		(pin "DP" bidirectional
 			(at 185.42 96.52 180)
 			(effects
@@
 			)
 		)
-		(pin "D-" bidirectional
+		(pin "DN" bidirectional
 			(at 185.42 99.06 180)
 			(effects
@@
 				)
 			)
+		)
+	)
+	(sheet
+		(at 196.85 124.46)
+		(size 74.93 31.75)
+		(exclude_from_sim no)
+		(in_bom yes)
+		(on_board yes)
+		(dnp no)
+		(fields_autoplaced yes)
+		(stroke
+			(width 0.1524)
+			(type solid)
+		)
+		(fill
+			(color 0 0 0 0.0000)
+		)
+		(property "Sheetname" "trou_fixation"
+			(at 196.85 123.7484 0)
+			(effects
+				(font
+					(size 1.27 1.27)
+				)
+				(justify left bottom)
+			)
+		)
+		(property "Sheetfile" "trou_fixation.kicad_sch"
+			(at 196.85 156.7946 0)
+			(effects
+				(font
+					(size 1.27 1.27)
+				)
+				(justify left top)
+			)
+		)
+		(property "Field2" ""
+			(at 196.85 124.46 0)
+			(effects
+				(font
+					(size 1.27 1.27)
+				)
+			)
+		)
+		(instances
+			(project "PCB_Casque"
+				(path "/dd9a0253-5793-4002-9ba2-74fe57888e3b"
+					(page "12")
+				)
+			)
