File: PCB_Casque/USB_c.kicad_sch (KiCad schematic)
At the start: 3 parts, among them J1 USB_C_Receptacle_USB2.0_16P

Commit message: ajout du PCB version final + elt du design
Connections:
- net D+ renamed DP
- net D- renamed DN
Changed lines of the file:
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@@
 		)
 	)
-	(hierarchical_label "D-"
+	(hierarchical_label "DN"
 		(shape output)
 		(at 149.86 82.55 0)
@@
 		)
 	)
-	(hierarchical_label "D+"
+	(hierarchical_label "DP"
 		(shape output)
 		(at 146.05 87.63 0)
